File: ComboFlex.kicad_sch (KiCad schematic)
At the start: 0 parts

Commit message: Initial NAND implementation
Parts:
- added C1, C2: 0.1uF, symbol Device:C_Small
- added C3: 1uF, symbol Device:C_Small
- added J1, J10, J11, J12, J13, J14, J15, J16, J17, J2, J3, J4, J5, J6, J7, J8, J9: Conn_01x01, symbol Connector_Generic:Conn_01x01
- added R1: 1k, symbol Device:R_Small
- added U1: ~, Package_SO:TSOP-I-48_18.4x12mm_P0.5mm, symbol ComboFlex:WiiNAND
Connections:
- new net: J9.1 (Pin_1), U1.19 (~{WP})
- new net: J7.1 (Pin_1), U1.17 (ALE)
- new net: J16.1 (Pin_1), U1.43 (I/O_6)
- new net: J8.1 (Pin_1), U1.18 (~{WE})
- new net: J14.1 (Pin_1), U1.41 (I/O_4)
- new net: J5.1 (Pin_1), U1.10 (EX2)
- new net: J6.1 (Pin_1), U1.16 (CLE)
- new net: J10.1 (Pin_1), U1.29 (I/O_0)
- new net: J11.1 (Pin_1), U1.30 (I/O_1)
- new net: J12.1 (Pin_1), U1.31 (I/O_2)
- new net: J13.1 (Pin_1), U1.32 (I/O_3)
- new net: J15.1 (Pin_1), U1.42 (I/O_5)
- new net: J17.1 (Pin_1), U1.44 (I/O_7)
- new net: J1.1 (Pin_1), U1.6 (EX1)
- new net: J2.1 (Pin_1), R1.2, U1.7 (~{R/B})
- new net: J3.1 (Pin_1), U1.8 (~{RE})
- new net: J4.1 (Pin_1), U1.9 (~{CE})
- new net +3.3V: C1.1, C2.1, C3.1, R1.1, U1.12 (VCC1), U1.37 (VCC2)
- new net GND: C1.2, C2.2, C3.2, U1.13 (VSS1), U1.36 (VSS2)

Commit message: Schematic mostly complete
Parts:
- added C10, C11, C12, C13, C14, C15, C16, C17, C9: 0.1uF, Capacitor_SMD:C_0402_1005Metric, symbol Device:C_Small
- added C4, C5: 5pF, Capacitor_SMD:C_0402_1005Metric, symbol Device:C_Small
- added C6: 100nF, Capacitor_SMD:C_0402_1005Metric, symbol Device:C_Small
- added C7, C8: 1uF, Capacitor_SMD:C_0402_1005Metric, symbol Device:C_Small
- added D1: D_Small, Diode_SMD:D_0603_1608Metric, symbol Device:D_Small
- added D2: BAT54XV2T1G, Diode_SMD:D_SOD-523, symbol Diode:MM5Zxx
- added J18: Conn_01x06_Pin, comboflex:wififlex, symbol Connector_Generic:Conn_01x06
- added J19: Conn_01x20_Pin, Connector_Molex:Molex_SlimStack_52991-0208_2x10_P0.50mm_Vertical, symbol Connector_Generic:Conn_01x20
- added J20: 505278-1933, 5052781933, symbol SamacSys_Parts:505278-1933
- added JP1: SolderJumper_2_Open, Jumper:SolderJumper-2_P1.3mm_Open_RoundedPad1.0x1.5mm, symbol Jumper:SolderJumper_2_Open
- added R2: 1k, Resistor_SMD:R_0402_1005Metric, symbol Device:R_Small
- added R3, R9: 4.7k, Resistor_SMD:R_0402_1005Metric, symbol Device:R_Small
- added R4, R5: 10k, Resistor_SMD:R_0402_1005Metric, symbol Device:R_Small
- added R6: 100K, Resistor_SMD:R_0402_1005Metric, symbol Device:R_Small
- added R7: 330, Resistor_SMD:R_0402_1005Metric, symbol Device:R_Small
- added R8: 0, Resistor_SMD:R_0402_1005Metric, symbol Device:R_Small
- added TP1: BATT, TestPoint:TestPoint_Pad_D1.0mm, symbol Connector:TestPoint
- added TP10, TP11, TP12: TestPoint, TestPoint:TestPoint_Pad_D1.5mm, symbol Connector:TestPoint
- added TP13, TP16: TestPoint, TestPoint:TestPoint_Pad_D1.0mm, symbol Connector:TestPoint
- added TP14, TP15, TP17, TP18, TP19, TP20: TestPoint, SamacSys_Parts:TestPoint_Pad_D0.75mm, symbol Connector:TestPoint
- added TP2: DATA0, Wii:TestPoint_THTPad_D0.5mm_Drill0.35mm, symbol Connector:TestPoint
- added TP3: DATA1, Wii:TestPoint_THTPad_D0.5mm_Drill0.35mm, symbol Connector:TestPoint
- added TP4: DATA2, Wii:TestPoint_THTPad_D0.5mm_Drill0.35mm, symbol Connector:TestPoint
- added TP5: DATA3, Wii:TestPoint_THTPad_D0.5mm_Drill0.35mm, symbol Connector:TestPoint
- added TP6: U10, TestPoint:TestPoint_Pad_D1.0mm, symbol Connector:TestPoint
- added TP7: U10, Wii:TestPoint_THTPad_D0.5mm_Drill0.35mm, symbol Connector:TestPoint
- added TP8: 3.3V, TestPoint:TestPoint_Pad_D1.0mm, symbol Connector:TestPoint
- added TP9: GND, Wii:TestPoint_THTPad_D0.5mm_Drill0.35mm, symbol Connector:TestPoint
- added U2: Wii-MX, Package_SO:SOIC-28W_7.5x17.9mm_P1.27mm, symbol Wii:Wii-MX
- added U3: ~, Package_TO_SOT_SMD:SOT-23-5, symbol Wii:U10
- added U4: TPS7A0512PDBZR, Package_TO_SOT_SMD:SOT-23, symbol Regulator_Linear:AP2127N-1.2
- added U5: XC3S200A-4VQG100C, QFP50P1600X1600X120-100N, symbol SamacSys_Parts:XC3S200A-4VQG100C
- added U6: AT25SF041B-MAHD-T, SON50P300X200X60-9N-D, symbol SamacSys_Parts:AT25SF041B-MAHD-T
- added Y1: 32.768kHz, Crystal:Crystal_SMD_2012-2Pin_2.0x1.2mm, symbol Device:Crystal
Connections:
- net +3.3V: now also C14.1, C15.1, C16.1, C17.1, C6.2, J19.11 (Pin_11), J19.12 (Pin_12), JP1.2 (B), R3.1, R8.1, R9.2, TP11.1, TP8.1, U2.17 (VDD), U2.24 (VDD), U2.25 (VDD), U2.27 (VDD), U3.5 (3.3V), U5.11 (VCCO_3), U5.22 (VCCAUX_1), U5.25 (IO_L01N_2/M0), U5.26 (VCCO_2_1), U5.29 (IO_L03N_2/VS2), U5.30 (IO_L04P_2/VS1), U5.31 (IO_L04N_2/VS0), U5.45 (VCCO_2_2), U5.55 (VCCAUX_2), U5.67 (VCCO_1), U5.68 (IP_1/VREF_1), U5.70 (IO_L05P_1), U5.79 (VCCO_0_1), U5.92 (VCCAUX_3), U5.96 (VCCO_0_2)
- net GND: now also C10.2, C11.2, C12.2, C13.2, C14.2, C15.2, C16.2, C17.2, C4.1, C5.1, C6.1, C7.2, C8.2, C9.2, J19.1 (Pin_1), J19.13 (Pin_13), J19.15 (Pin_15), J19.18 (Pin_18), J19.20 (Pin_20), J19.4 (Pin_4), J19.6 (Pin_6), J19.8 (Pin_8), J20.12, J20.15, J20.18, J20.3, J20.9, J20.MP1, J20.MP2, R7.2, TP10.1, TP9.1, U2.16 (GND), U2.4 (GND), U3.1 (GND), U3.2 (GND), U3.3 (GND), U4.1 (GND), U5.14 (GND_2), U5.18 (GND_3), U5.23 (IO_L01P_2/M1), U5.24 (IO_L02P_2/M2), U5.42 (GND_4), U5.47 (GND_5), U5.58 (GND_6), U5.63 (GND_7), U5.69 (GND_8), U5.74 (GND_9), U5.8 (GND_1), U5.80 (GND_10), U5.87 (GND_11), U5.91 (GND_12), U5.95 (GND_13), U6.4 (GND), U6.9 (EP)
- new net: TP6.1, TP7.1, U3.4 (RST)
- new net: R9.1, U5.48 (IO_L10P_2/INIT_B)
- new net: C4.2, U2.23 (X_1), Y1.2
- new net: R3.2, U5.100 (PROG_B)
- new net: R7.1, U5.54 (DONE)
- new net: C13.1, R6.1, R8.2, U6.3 (~{WP_(IO2})), U6.7 (~{HOLD_(IO3})), U6.8 (VCC)
- new net: C5.2, U2.22 (X_2), Y1.1
- new net: D1.1 (K), U2.26 (BATT)
- new net: J20.4, R5.2
- new net: D1.2 (A), R2.1
- new net: J18.1 (Pin_1), J19.16 (Pin_16)
- new net: J18.2 (Pin_2), J19.17 (Pin_17)
- new net: J18.3 (Pin_3), J19.19 (Pin_19)
- new net: J18.4 (Pin_4), J19.5 (Pin_5)
- new net: J18.5 (Pin_5), J19.3 (Pin_3)
- new net: J18.6 (Pin_6), J19.2 (Pin_2)
- new net: D2.1 (K), J20.2
- new net: J20.5, R4.2
- new net +1V2: C10.1, C11.1, C12.1, C8.1, C9.1, U4.2 (VO), U5.17 (VCCINT_1), U5.38 (VCCINT_2), U5.66 (VCCINT_3), U5.81 (VCCINT_4)
- new net +1V8: C7.1, TP12.1, U4.3 (VI)
- new net +5V: D2.2 (A), R4.1, R5.1, TP13.1
- new net 54MHz: U5.43 (IO_L09P_2/GCLK0)
- new net BATT: R2.2, TP1.1
- new net C: U5.41 (IO_L08N_2/GCLK15)
- new net CLK: TP20.1, U5.53 (IO_L12N_2/CCLK), U6.6 (SCK)
- new net CS: R6.2, TP17.1, U5.27 (IO_L02N_2/CSO_B), U6.1 (~{CS})
- new net CSEL: U5.5 (IO_L02P_3)
- new net D: U5.40 (O_L08P_2/GCLK14)
- new net D0: U5.6 (IO_L02N_3)
- new net D1: U5.7 (IP_3/VREF_3)
- new net D2: U5.9 (IO_L03P_3/LHCLK0)
- new net D3: U5.10 (IO_L03N_3/LHCLK1)
- new net D4: U5.12 (IO_L04P_3/LHCLK2)
- new net D5: U5.13 (IO_L04N_3/IRDY2/LHCLK3)
- new net D6: U5.15 (IO_L05P_3/TRDY2/LHCLK6)
- new net D7: U5.16 (IO_L05N_3/LHCLK7)
- new net DATA0: TP2.1, U2.11 (DATA0)
- new net DATA1: TP3.1, U2.12 (DATA1)
- new net DATA2: TP4.1, U2.13 (DATA2)
- new net DATA3: TP5.1, U2.14 (DATA3)
- new net GCC: TP16.1, U5.73 (IO_L06N_1)
- new net MISO: TP19.1, U5.51 (IO_L12P_2/D0/DIN/MISO), U6.2 (SO_(IO1))
- new net MODE: JP1.1 (A)
- new net MOSI: TP18.1, U5.46 (IO_2/MOSI/CSI_B), U6.5 (SI_(IO0))
- new net SCL: TP15.1
- new net SDA: TP14.1
- new net TMDS0+: J20.13, U5.84 (IO_L02N_0/GCLK5)
- new net TMDS0-: J20.11, U5.83 (IO_L02P_0/GCLK4)
- new net TMDS1+: J20.16, U5.89 (IO_L04N_0/GCLK9)
- new net TMDS1-: J20.14, U5.88 (IO_L04P_0/GCLK8)
- new net TMDS2+: J20.19, U5.94 (IO_L05N_0)
- new net TMDS2-: J20.17, U5.93 (IO_L05P_0)
- new net TMDSClk+: J20.10, U5.78 (IO_L01N_0)
- new net TMDSClk-: J20.8, U5.77 (IO_L01P_0/VREF_0)
- new net W: U5.39 (IP_2/VREF_2)
- no-connect marks 0 -> 44
Other:
- note added: "FujiFlex"
- note added: "HDMI Pin 1"
- note added: "HDMI Pin 19"
- note added: "NAND relocation"
- note added: "WiFi flex"
- note added: "mxHound"
- note added: "x4 0.1uF"
- moved on the sheet: C1, C2, C3, J1, J10, J11, J12, J13, J14, J15, J16, J17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

Commit message: PCB work, NAND portion mostly complete
Parts:
- removed Y1: 32.768kHz, Crystal:Crystal_SMD_2012-2Pin_2.0x1.2mm, symbol Device:Crystal
- added BT1: CR2032, Battery:BatteryHolder_Keystone_1058_1x2032, symbol Device:Battery_Cell
- added TP21: RESET, comboflex:TestPoint_THTPad_D0.5mm_Drill0.35mm, symbol Connector:TestPoint
- added TP22: RESET, TestPoint:TestPoint_Pad_D1.0mm, symbol Connector:TestPoint
- added X1: 32.768kHz, Crystal:Crystal_SMD_Abracon_ABS25-4Pin_8.0x3.8mm, symbol Device:Crystal_GND23
- C1, C2, C3: footprint (none) -> Capacitor_SMD:C_0402_1005Metric
- J1, J10, J11, J12, J13, J14, J15, J16, J17, J2, J3, J4, J5, J6, J7, J8, J9: footprint (none) -> comboflex:wii-single-via-0.45mm
- R1: footprint (none) -> Resistor_SMD:R_0402_1005Metric
- TP2, TP3, TP4, TP5, TP7, TP9: footprint Wii:TestPoint_THTPad_D0.5mm_Drill0.35mm -> comboflex:TestPoint_THTPad_D0.5mm_Drill0.35mm
- U1: footprint Package_SO:TSOP-I-48_18.4x12mm_P0.5mm -> comboflex:Wii-TSOP48-trimmed
- U5: footprint QFP50P1600X1600X120-100N -> comboflex:QFP50P1600X1600X120-100N
Connections:
- net BATT: now also BT1.1 (+)
- net GND: now also BT1.2 (-), X1.2, X1.3
- net at C4.2, U2.23 (X_1): now also X1.4
- net at C5.2, U2.22 (X_2): now also X1.1
- new net Wii_RESET: TP21.1, TP22.1
Other:
- moved on the sheet: TP2, TP3, TP4, TP5

Commit message: Nearing completion
Parts:
- removed X1: 32.768kHz, Crystal:Crystal_SMD_Abracon_ABS25-4Pin_8.0x3.8mm, symbol Device:Crystal_GND23
- added TP23: SoftEcho, comboflex:TestPoint_THTPad_D0.5mm_Drill0.35mm, symbol Connector:TestPoint
- added TP24: SoftEcho, comboflex:TestPoint_Pad_D0.75mm, symbol Connector:TestPoint
- added TP25: SoftShut, comboflex:TestPoint_THTPad_D0.5mm_Drill0.35mm, symbol Connector:TestPoint
- added TP26: SoftShut, comboflex:TestPoint_Pad_D0.75mm, symbol Connector:TestPoint
- added Y1: 32.768kHz, Crystal:Crystal_SMD_2012-2Pin_2.0x1.2mm, symbol Device:Crystal
- J20: footprint 5052781933 -> comboflex:5052781933
- TP14, TP15, TP17, TP18, TP19, TP20: footprint SamacSys_Parts:TestPoint_Pad_D0.75mm -> comboflex:TestPoint_Pad_D0.75mm
- TP22, TP6: footprint TestPoint:TestPoint_Pad_D1.0mm -> comboflex:TestPoint_Pad_D0.75mm
- U6: footprint SON50P300X200X60-9N-D -> Package_SON:SON-8-1EP_3x2mm_P0.5mm_EP1.4x1.6mm
Connections:
- net at C4.2, U2.23 (X_1): now also Y1.2
- net at C5.2, U2.22 (X_2): now also Y1.1
- new net SoftEcho: TP23.1, TP24.1
- new net SoftShut: TP25.1, TP26.1

Commit message: More adjustments
Parts:
- removed TP8: 3.3V, TestPoint:TestPoint_Pad_D1.0mm, symbol Connector:TestPoint
- added TP27: GND, TestPoint:TestPoint_Pad_D1.0mm, symbol Connector:TestPoint
Connections:
- net GND: now also TP27.1
Changed lines of the file:
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@@
 	)
 	(symbol
-		(lib_id "Connector:TestPoint")
-		(at 74.93 77.47 180)
-		(unit 1)
-		(exclude_from_sim no)
-		(in_bom yes)
-		(on_board yes)
-		(dnp no)
-		(fields_autoplaced yes)
-		(property "Reference" "TP8"
-			(at 77.47 79.502 0)
-			(effects
-				(font
-					(size 1.27 1.27)
-				)
-				(justify right)
-			)
-		)
-		(property "Value" "3.3V"
-			(at 77.47 82.042 0)
-			(effects
-				(font
-					(size 1.27 1.27)
-				)
-				(justify right)
-			)
-		)
-		(property "Footprint" "TestPoint:TestPoint_Pad_D1.0mm"
-			(at 69.85 77.47 0)
-			(effects
-				(font
-					(size 1.27 1.27)
-				)
-				(hide yes)
-			)
-		)
-		(property "Datasheet" "~"
-			(at 69.85 77.47 0)
-			(effects
-				(font
-					(size 1.27 1.27)
-				)
-				(hide yes)
-			)
-		)
-		(property "Description" ""
-			(at 74.93 77.47 0)
-			(effects
-				(font
-					(size 1.27 1.27)
-				)
-				(hide yes)
-			)
-		)
-		(pin "1"
-		)
-		(instances
-			(project "ComboFlex"
-				(path "/e2d101d3-bf42-4f61-a881-d4588bf3891c"
-					(reference "TP8")
-					(unit 1)
-				)
-			)
-		)
-	)
-	(symbol
 		(lib_id "power:GND")
 		(at 24.13 44.45 0)
@@
 	)
 	(symbol
+		(lib_id "Connector:TestPoint")
+		(at 77.47 104.14 0)
+		(unit 1)
+		(exclude_from_sim no)
+		(in_bom yes)
+		(on_board yes)
+		(dnp no)
+		(fields_autoplaced yes)
+		(property "Reference" "TP27"
+			(at 80.01 99.568 0)
+			(effects
+				(font
+					(size 1.27 1.27)
+				)
+				(justify left)
+			)
+		)
+		(property "Value" "GND"
+			(at 80.01 102.108 0)
+			(effects
+				(font
+					(size 1.27 1.27)
+				)
+				(justify left)
+			)
+		)
+		(property "Footprint" "TestPoint:TestPoint_Pad_D1.0mm"
+			(at 82.55 104.14 0)
+			(effects
+				(font
+					(size 1.27 1.27)
+				)
+				(hide yes)
+			)
+		)
+		(property "Datasheet" "~"
+			(at 82.55 104.14 0)
+			(effects
+				(font
+					(size 1.27 1.27)
+				)
+				(hide yes)
+			)
+		)
+		(property "Description" ""
+			(at 77.47 104.14 0)
+			(effects
+				(font
+					(size 1.27 1.27)
+				)
+				(hide yes)
+			)
+		)
+		(pin "1"
+		)
+		(instances
+			(project "ComboFlex"
+				(path "/e2d101d3-bf42-4f61-a881-d4588bf3891c"
+					(reference "TP27")
+					(unit 1)
+				)
+			)
+		)
+	)
+	(symbol
 		(lib_id "power:+3.3V")
 		(at 85.09 77.47 0)
@@
 	)
 	(symbol
-		(lib_id "power:+3.3V")
-		(at 74.93 77.47 0)
-		(unit 1)
-		(exclude_from_sim no)
-		(in_bom yes)
-		(on_board yes)
-		(dnp no)
-		(fields_autoplaced yes)
-		(property "Reference" "#PWR012"
-			(at 74.93 81.28 0)
-			(effects
-				(font
-					(size 1.27 1.27)
-				)
-				(hide yes)
-			)
-		)
-		(property "Value" "+3.3V"
-			(at 74.93 72.39 0)
-			(effects
-				(font
-					(size 1.27 1.27)
-				)
-			)
-		)
-		(property "Footprint" ""
-			(at 74.93 77.47 0)
-			(effects
-				(font
-					(size 1.27 1.27)
-				)
-				(hide yes)
-			)
-		)
-		(property "Datasheet" ""
-			(at 74.93 77.47 0)
-			(effects
-				(font
-					(size 1.27 1.27)
-				)
-				(hide yes)
-			)
-		)
-		(property "Description" ""
-			(at 74.93 77.47 0)
-			(effects
-				(font
-					(size 1.27 1.27)
-				)
-				(hide yes)
-			)
-		)
-		(pin "1"
-		)
-		(instances
-			(project "ComboFlex"
-				(path "/e2d101d3-bf42-4f61-a881-d4588bf3891c"
-					(reference "#PWR012")
-					(unit 1)
-				)
-			)
-		)
-	)
-	(symbol
 		(lib_name "Conn_01x01_1")
 		(lib_id "Connector_Generic:Conn_01x01")
@@
 					(unit 1)
 				)
+			)
+		)
+	)
+	(symbol
+		(lib_id "power:GND")
+		(at 77.47 104.14 0)
+		(unit 1)
+		(exclude_from_sim no)
+		(in_bom yes)
+		(on_board yes)
+		(dnp no)
+		(fields_autoplaced yes)
+		(property "Reference" "#PWR049"
+			(at 77.47 110.49 0)
+			(effects
+				(font
+					(size 1.27 1.27)
+				)
+				(hide yes)
+			)
+		)
+		(property "Value" "GND"
+			(at 77.47 109.22 0)
+			(effects
+				(font
+					(size 1.27 1.27)
+				)
+			)
+		)
+		(property "Footprint" ""
+			(at 77.47 104.14 0)
+			(effects
+				(font
+					(size 1.27 1.27)
+				)
+				(hide yes)
+			)
+		)
+		(property "Datasheet" ""
+			(at 77.47 104.14 0)
+			(effects
+				(font
+					(size 1.27 1.27)
+				)
+				(hide yes)
+			)
+		)
+		(property "Description" ""
+			(at 77.47 104.14 0)
+			(effects
+				(font
+					(size 1.27 1.27)
+				)
+				(hide yes)
+			)
+		)
+		(pin "1"
+		)
+		(instances
+			(project "ComboFlex"
+				(path "/e2d101d3-bf42-4f61-a881-d4588bf3891c"
+					(reference "#PWR049")
+					(unit 1)
+				)
